File: microdrill/schematics/drill.kicad_pcb (KiCad board)
At the start: 2 copper layers, 11 parts, among them P1 CONN_2, P2 CONN_2, P3 CONN_2, Q1 MOS_N, U1 LM555N

Commit message: Testet automatic drill speed management
Parts:
- removed Q1: MOS_N, TO220
- removed RV1: POT, PIN_ARRAY_3X1
- added C2: 104, SM0603_Capa, F.Cu at (239.4, 72.8)
- added C3: 104, SM0603_Capa, F.Cu at (254.3, 72.8)
- added C4: 0.1u, SM0603, F.Cu at (257.2, 72.8)
- added C5: 47u, SM1206, F.Cu at (229.0, 73.4)
- added C6: 47u, SM1206POL, F.Cu at (223.0, 73.4)
- added D1: LED, LED-0603, F.Cu at (260.0, 72.6)
- added D2: LED, LED-0603, F.Cu at (262.8, 72.6)
- added D3: DIODESCH, D4, F.Cu at (215.9, 63.2)
- added K1: POWER, PIN_ARRAY_3X1, F.Cu at (205.1, 73.4)
- added P4: Slide, SIL-2, F.Cu at (211.7, 73.5)
- added P5: CONN_14, SIL-14, F.Cu at (243.3, 53.8)
- added P6: CONN_5, SIL-5, F.Cu at (204.6, 63.2)
- added P7: CONN_2, SIL-2, F.Cu at (217.3, 73.5)
- added R5: 1R, R4, F.Cu at (261.2, 63.0)
- added R6: 1R, R4, F.Cu at (195.2, 73.3)
- added R7: 1R, R4, F.Cu at (249.4, 63.0)
- added SW1: DRILL, 2PIN_6mm, F.Cu at (254.9, 32.6)
- added SW2: UP, 2PIN_6mm, F.Cu at (254.9, 45.8)
- added SW3: DOWN, 2PIN_6mm, F.Cu at (211.2, 45.8)
- added SW4: SW_PUSH, 2PIN_6mm, F.Cu at (211.2, 32.6)
- added U2: LM1117MPX-3.3, SOT223, F.Cu at (193.0, 67.3)
- C1: footprint C1 -> SM1206
- P1: value CONN_2 -> CONN_14; footprint SIL-2 -> SIL-14
- P2: value CONN_2 -> CONN_4; footprint SIL-2 -> SIL-4
- P3: value CONN_2 -> Stepper; footprint SIL-2 -> SIL-4
- R1: value 10k -> 1k; footprint SM0805 -> SM0603
- R2: footprint SM0805 -> SM0603
- R3: value 1R -> 10k; footprint R3 -> SM0603
- R4: value 1R -> 47k; footprint R3 -> SM0603
- U1: value LM555N -> STM8S105K4T6C
- moved U1 110.1 mm to (266.6, 57.0)
- moved R3 108.6 mm to (245.4, 72.8)
- moved R2 107.4 mm to (251.2, 72.8)
- moved R1 101.4 mm to (248.3, 72.8)
- moved P2 101.0 mm to (238.1, 63.2)
- moved R4 97.7 mm to (242.3, 72.8)
- moved P3 86.0 mm to (227.6, 63.2)
- moved C1 85.3 mm to (234.9, 73.4)
- moved P1 74.1 mm to (207.3, 53.8)
Connections:
- C1 pad 1: N-000001 -> GND
- C1 pad 2: GND -> N-0000031
- P1 pad 1: +12V -> +3.3V
- P1 pad 2: N-000006 -> GND
- P2 pad 1: GND -> +3.3V
- P2 pad 2: VCC -> /SWIM/PD1
- P3 pad 1: GND -> N-0000014
- P3 pad 2: +12V -> N-000005
- R1 pad 1: VCC -> N-0000040
- R1 pad 2: N-000001 -> /PC2
- R2 pad 1: N-000004 -> N-0000039
- R2 pad 2: N-000001 -> GND
- R3 pad 1: N-000006 -> +3.3V
- R3 pad 2: N-000007 -> /NRST
- R4 pad 1: N-000006 -> /Drill motor/Sence
- R4 pad 2: N-000007 -> N-0000041
- U1 pad 1: GND -> /NRST
- U1 pad 2: N-000006 -> /OSC1IN
- U1 pad 3: N-000009 -> /OSC2IN
- U1 pad 4: VCC -> GND
- U1 pad 5: N-000008 -> N-0000031
- U1 pad 6: N-000006 -> +3.3V
- U1 pad 7: N-000004 -> +3.3V
- U1 pad 8: VCC -> /Drill motor/Sence
