File: microdrill/schematics/MCU_module.kicad_pcb (KiCad board)
At the start: 2 copper layers, 0 parts

Commit message: started voltmeter hacking
Parts:
- added BTN1: CONN_1, PINTST, F.Cu at (123.7, 79.5)
- added BTN2: CONN_1, PINTST, F.Cu at (121.2, 79.5)
- added C4: 0.1u, SM0603, B.Cu at (100.1, 98.0)
- added C5: 47u, SM1206POL, B.Cu at (102.1, 102.9)
- added C6: 0.1u, SM0603, B.Cu at (112.8, 102.6)
- added DA1: L9110, so-8, B.Cu at (132.1, 96.0)
- added DA2: L9110, so-8, B.Cu at (132.1, 90.2)
- added DA3: L9110, so-8, F.Cu at (105.7, 89.9)
- added DOWN1: CONN_1, PINTST, F.Cu at (131.3, 79.5)
- added DRILL+1: CONN_1, PINTST, F.Cu at (96.3, 91.4)
- added DRILL-1: CONN_1, PINTST, F.Cu at (138.2, 101.3)
- added DRILLSW1: CONN_1, PINTST, F.Cu at (126.2, 79.5)
- added GND1: CONN_1, PINTST, F.Cu at (96.3, 102.4)
- added K1: POWER, PIN_ARRAY_3X1, F.Cu at (96.3, 96.8)
- added P3: Stepper, PIN_ARRAY_4x1, B.Cu at (138.2, 93.0)
- added P4: Slide, PIN_ARRAY_2X1, F.Cu at (96.3, 86.9)
- added POT1: CONN_1, PINTST, F.Cu at (118.6, 110.5)
- added R4: 47k, SM0603, B.Cu at (117.6, 102.6)
- added R5: 0.33R, r_2512, B.Cu at (118.4, 96.8)
- added U2: LM1117MPX-3.3, SOT223, B.Cu at (105.2, 94.0)
- added UP1: CONN_1, PINTST, F.Cu at (128.8, 79.5)
- added VT1: S8205A, TSSOP-8, F.Cu at (134.8, 98.8)
- added X1: STM8S105BOARD, devboard_pins-9-14, F.Cu at (117.3, 95.0)
Routing:
- net GND: track 0.00 -> 82.4 mm, vias 0 -> 1
- net +5V: track 0.00 -> 68.3 mm, vias 0 -> 1
- net N-0000038: track 0.00 -> 30.6 mm, vias 0 -> 1
- net /PB3: track 0.00 -> 22.3 mm
- net /PB2: track 0.00 -> 19.1 mm
- net /PB1: track 0.00 -> 13.6 mm
- net +3.3V: track 0.00 -> 13.4 mm
- net /PB0: track 0.00 -> 12.3 mm
- net /PD2: track 0.00 -> 10.7 mm, vias 0 -> 1
- net /Drill motor/PWM_in: track 0.00 -> 10.4 mm, vias 0 -> 1
- net /Drill motor/DRILL-: track 0.00 -> 9.52 mm, vias 0 -> 1
- net N-0000017: track 0.00 -> 8.58 mm, vias 0 -> 1
- net N-0000016: track 0.00 -> 7.60 mm, vias 0 -> 1
- net /PD3: track 0.00 -> 7.58 mm, vias 0 -> 1
- net /Drill motor/Sence: track 0.00 -> 7.11 mm
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- added copper zone on B.Cu, net GND
- added copper zone on F.Cu, net GND
Other:
- board outline added: 47 x 34 mm
- net class Default: via_dia 0.889 -> 1; via_drill 0.635 -> 0.6
- net class high-power added: clearance 0.254, trace_width 1, via_dia 1.5, via_drill 0.8
- net class power added: clearance 0.254, trace_width 0.5, via_dia 1.3, via_drill 0.8
- board text added: "1"
- board text added: "12"
- board text added: "5"
- board text added: "BTN2,BTN1,PEDAL,UP,DOWN"
- board text added: "DRL-"
- board text added: "GND"
- board text added: "POT"
- board text added: "STPR"
- board text added: "Tray"
