File: microdrill/schematics/MCU_module.sch (KiCad schematic (older format))
At the start: 26 parts, among them K1 POWER, P1 CONN_14, P2 CONN_4, P3 Stepper, P4 Slide, P5 CONN_14, P6 CONN_5, SW1 SW_PUSH, U1 STM8S105K4T6C, U2 LM1117MPX-3.3

Commit message: Testet automatic drill speed management
Parts:
- gave numbers to parts that had none: 3
- renumbered SW1 to SW4
Changed lines of the file:
@@
 Sheet 1 2
 Title ""
-Date "17 aug 2014"
+Date "19 aug 2014"
 Rev ""
 Comp ""
@@
 	6500 3850 6500 4050
 $Comp
-L SW_PUSH SW1
+L SW_PUSH SW4
 U 1 1 52FB0F3B
 P 6500 3550
-F 0 "SW1" H 6650 3660 50  0000 C CNN
+F 0 "SW4" H 6650 3660 50  0000 C CNN
 F 1 "SW_PUSH" H 6500 3470 50  0000 C CNN
 F 2 "" H 6500 3550 60  0000 C CNN
@@
 	5700 8450 3550 8450
 $Comp
-L SW_PUSH SW?
+L SW_PUSH SW2
 U 1 1 53F12B09
 P 4150 8250
-F 0 "SW?" H 4300 8360 50  0000 C CNN
+F 0 "SW2" H 4300 8360 50  0000 C CNN
 F 1 "UP" H 4150 8170 50  0000 C CNN
 F 2 "~" H 4150 8250 60  0000 C CNN
@@
 $EndComp
 $Comp
-L SW_PUSH SW?
+L SW_PUSH SW3
 U 1 1 53F12B1C
 P 5050 8250
-F 0 "SW?" H 5200 8360 50  0000 C CNN
+F 0 "SW3" H 5200 8360 50  0000 C CNN
 F 1 "DOWN" H 5050 8170 50  0000 C CNN
 F 2 "~" H 5050 8250 60  0000 C CNN
@@
 	4450 8250 4750 8250
 $Comp
-L GND #PWR?
+L GND #PWR028
 U 1 1 53F12BC1
 P 4600 8350
-F 0 "#PWR?" H 4600 8350 30  0001 C CNN
+F 0 "#PWR028" H 4600 8350 30  0001 C CNN
 F 1 "GND" H 4600 8280 30  0001 C CNN
 F 2 "" H 4600 8350 60  0000 C CNN
@@
 PC3
 $Comp
-L SW_PUSH SW?
+L SW_PUSH SW1
 U 1 1 53F13089
 P 1650 6750
-F 0 "SW?" H 1800 6860 50  0000 C CNN
+F 0 "SW1" H 1800 6860 50  0000 C CNN
 F 1 "DRILL" H 1650 6670 50  0000 C CNN
 F 2 "~" H 1650 6750 60  0000 C CNN
@@
 $EndComp
 $Comp
-L GND #PWR?
+L GND #PWR029
 U 1 1 53F130B8
 P 1950 6950
-F 0 "#PWR?" H 1950 6950 30  0001 C CNN
+F 0 "#PWR029" H 1950 6950 30  0001 C CNN
 F 1 "GND" H 1950 6880 30  0001 C CNN
 F 2 "" H 1950 6950 60  0000 C CNN

Commit message: Modified some code on "frum" and "microdrill"
Parts:
- added RV1: POT, symbol POT
- added SW5: UP, ~, symbol SW_PUSH
- added SW6: DOWN, ~, symbol SW_PUSH
- SW2: value UP -> BTN1
- SW3: value DOWN -> BTN2
Connections:
- wire segments 95 -> 100
Other:
- note added: ""DRILL" is foot-switch.\nPress it to move drill down,\nrelease to return it to start position.\nDouble-click turns drill motor on/off.\n"
- note added: "All MCU inputs connected to switches\nshould be in "pull-up input" mode."
- note added: "BTN1"
- note added: "BTN2"
- note added: "Drill PWM"
- note added: "Drill SW"
- note added: "Drill sense"
- note added: "LED onbrd"
- note added: "Rvar"
- note added: "Stepper phases"
- note added: "Tray Down"
- note added: "Tray Up"
- note added: "Tray bridge"
- note added: "Two buttons on tray have following functionality:\nBTN1 - setup zero point (move slowly + set coordinate\n to 0 after footswitch released); next pressing returns\n device to normal state;\nBTN2 - switch between regulation of drill speed/stepper speed;\nBTN1+BTN2 (simultaneously) - move tray up/down.\n\n"volume" varistor allows to regulate motor speed.\nDefault is max drill speed, varistor regulat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"
- note added: "UART"

Commit message: started voltmeter hacking
Parts:
- removed C1: 1u, symbol C
- removed C2, C3: 104, symbol C
- removed D1, D2: LED, symbol LED
- removed P1, P5: CONN_14, symbol CONN_14
- removed P2: CONN_4, symbol CONN_4
- removed P6: CONN_5, symbol CONN_5
- removed R1, R2: 1k, symbol R
- removed R3: 10k, symbol R
- removed RV1: POT, symbol POT
- removed SW1: DRILL, ~, symbol SW_PUSH
- removed SW2: BTN1, ~, symbol SW_PUSH
- removed SW3: BTN2, ~, symbol SW_PUSH
- removed SW4: SW_PUSH, symbol SW_PUSH
- removed SW5: UP, ~, symbol SW_PUSH
- removed SW6: DOWN, ~, symbol SW_PUSH
- removed U1: STM8S105K4T6C, ~, symbol STM8S105K4T6C
- added BTN1, BTN2, DOWN1, DRILL+1, DRILL-1, DRILLSW1, GND1, POT1, UP1: CONN_1, symbol CONN_1
- added X1: stm8s105board, devboard_pins-9-14, symbol stm8s105board
Connections:
- net labels removed: 3.3V, 5.0V, RXD, TXD
- wire segments 100 -> 69
- no-connect marks 1 -> 12
Other:
- note added: ""DRILLSW" is foot-switch.\nPress it to move drill down,\nrelease to return it to start position.\nDouble-click turns drill motor on/off.\n"
- note added: "Drill motor + pedal"
- note added: "Tray"
- note removed: ""DRILL" is foot-switch.\nPress it to move drill down,\nrelease to return it to start position.\nDouble-click turns drill motor on/off.\n"
- note removed: "Drill motor"
- note removed: "STM8 board"
- note removed: "Slider (tray) motor"
- note removed: "USB <-> TTL"
