File: DRUM/schematics/drum.kicad_pcb (KiCad board)
At the start: 2 copper layers, 0 parts

Commit message: Modified some code on "frum" and "microdrill"
Parts:
- added C3: 100u, CP_5x11mm, F.Cu at (73.5, 29.0)
- added C4: 100u, CP_5x11mm, F.Cu at (79.1, 29.0)
- added DA1: TDA2822, DIP-8__300, F.Cu at (76.5, 42.9)
- added DD1: CD74HC154, DIP-24__300, F.Cu at (50.0, 43.9)
- added P10: CONN_1, SIL-1, F.Cu at (72.1, 34.8)
- added P11: CONN_1, SIL-1, F.Cu at (69.7, 26.0)
- added P12: CONN_1, SIL-1, F.Cu at (46.4, 56.5)
- added P13: CONN_1, SIL-1, F.Cu at (48.9, 56.5)
- added P15: CONN_1, SIL-1, F.Cu at (54.0, 56.5)
- added P16: CONN_1, SIL-1, F.Cu at (56.5, 56.5)
- added P18: CONN_1, SIL-1, F.Cu at (36.2, 26.0)
- added P19: CONN_1, SIL-1, F.Cu at (38.7, 26.0)
- added P20: CONN_1, SIL-1, F.Cu at (60.3, 35.1)
- added P21: CONN_1, SIL-1, F.Cu at (62.9, 35.1)
- added P22: CONN_1, SIL-1, F.Cu at (65.4, 35.1)
- added P23: CONN_1, SIL-1, F.Cu at (67.9, 35.1)
- added P24: CONN_1, SIL-1, F.Cu at (67.9, 37.6)
- added P25: CONN_1, SIL-1, F.Cu at (67.9, 40.1)
- added P26: CONN_1, SIL-1, F.Cu at (59.1, 26.0)
- added P27: CONN_1, SIL-1, F.Cu at (61.6, 26.0)
- added P28: CONN_1, SIL-1, F.Cu at (64.1, 26.0)
- added P29: CONN_1, SIL-1, F.Cu at (66.7, 26.0)
- added P7: CONN_10, SIL-10, B.Cu at (42.4, 37.7)
- added P8: CONN_1, SIL-1, F.Cu at (71.8, 51.7)
- added P9: CONN_1, SIL-1, F.Cu at (28.6, 51.6)
- added Q1: 2N7002, transistors_gaui-SOT23, F.Cu at (52.8, 33.8)
- added Q2: 2N7002, transistors_gaui-SOT23, F.Cu at (48.3, 33.9)
- added Q3: 2N7002, transistors_gaui-SOT23, F.Cu at (44.1, 34.0)
- added Q4: 2N7002, transistors_gaui-SOT23, F.Cu at (40.1, 34.2)
- added Q5: 2N7002, transistors_gaui-SOT23, F.Cu at (35.6, 34.2)
- added Q6: 2N7002, transistors_gaui-SOT23, F.Cu at (30.9, 34.2)
- added R1: 10k, SM0603, B.Cu at (75.1, 34.8)
- added R2: 10k, SM0603, B.Cu at (74.9, 54.4)
- added R3: 3.3k, SM0603, B.Cu at (76.6, 37.0)
- added R4: 10k, SM0603, B.Cu at (76.5, 49.9)
- added X1: STM8S105BOARD, devboard_pins-9-14, F.Cu at (50.2, 41.3)
Routing:
- net GND: track 0.00 -> 82.1 mm
- net VCC: track 0.00 -> 59.4 mm, vias 0 -> 3
- net /PC6: track 0.00 -> 47.8 mm
- net N-0000052: track 0.00 -> 25.4 mm
- net /PE5: track 0.00 -> 19.3 mm
- net N-0000017: track 0.00 -> 18.8 mm
- net /PD4: track 0.00 -> 18.4 mm
- net /DRUM/LED5: track 0.00 -> 12.6 mm
- net /DRUM/LED4: track 0.00 -> 11.7 mm
- net /DRUM/LED3: track 0.00 -> 11.6 mm
- net /DRUM/LED2: track 0.00 -> 11.6 mm
- net /PD3: track 0.00 -> 11.6 mm, vias 0 -> 1
- net /DRUM/SPEAKER: track 0.00 -> 10.1 mm
- net N-0000015: track 0.00 -> 9.63 mm
- net /PD2: track 0.00 -> 9.31 mm, vias 0 -> 1
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- added copper zone on B.Cu, net GND
- added copper zone on F.Cu, net GND
Other:
- board outline added: 57 x 34 mm
- net class Default: trace_width 0.254 -> 0.4; via_dia 0.889 -> 1; via_drill 0.635 -> 0.8
