File: DRUM/schematics/DRUM_itself.sch (KiCad schematic (older format))
At the start: 16 parts

Commit message: modified DRUM schematics
Parts:
- gave numbers to parts that had none: 16
Changed lines of the file:
@@
 LIBS:tda2822
 LIBS:CD74HC154
+LIBS:transistors_gaui
 LIBS:drum-cache
 EELAYER 27 0
@@
 Sheet 2 3
 Title ""
-Date "28 jul 2014"
+Date "20 sep 2014"
 Rev ""
 Comp ""
@@
 $EndDescr
 $Comp
-L SPEAKER SP?
+L SPEAKER SP1
 U 1 1 53D64216
 P 3950 1750
-F 0 "SP?" H 3850 2000 70  0000 C CNN
+F 0 "SP1" H 3850 2000 70  0000 C CNN
 F 1 "SPEAKER" H 3850 1500 70  0000 C CNN
 F 2 "" H 3950 1750 60  0000 C CNN
@@
 $EndComp
 $Comp
-L CRYSTAL X?
+L CRYSTAL X2
 U 1 1 53D64225
 P 3750 2950
-F 0 "X?" H 3750 3100 60  0000 C CNN
+F 0 "X2" H 3750 3100 60  0000 C CNN
 F 1 "CRYSTAL" H 3750 2800 60  0000 C CNN
 F 2 "" H 3750 2950 60  0000 C CNN
@@
 $EndComp
 $Comp
-L CRYSTAL X?
+L CRYSTAL X1
 U 1 1 53D64234
 P 3750 2500
-F 0 "X?" H 3750 2650 60  0000 C CNN
+F 0 "X1" H 3750 2650 60  0000 C CNN
 F 1 "CRYSTAL" H 3750 2350 60  0000 C CNN
 F 2 "" H 3750 2500 60  0000 C CNN
@@
 $EndComp
 $Comp
-L LED D?
+L LED D5
 U 1 1 53D6424D
 P 1900 3600
-F 0 "D?" H 1900 3700 50  0000 C CNN
+F 0 "D5" H 1900 3700 50  0000 C CNN
 F 1 "LED" H 1900 3500 50  0000 C CNN
 F 2 "" H 1900 3600 60  0000 C CNN
@@
 $EndComp
 $Comp
-L LED D?
+L LED D6
 U 1 1 53D6425A
 P 1900 3900
-F 0 "D?" H 1900 4000 50  0000 C CNN
+F 0 "D6" H 1900 4000 50  0000 C CNN
 F 1 "LED" H 1900 3800 50  0000 C CNN
 F 2 "" H 1900 3900 60  0000 C CNN
@@
 $EndComp
 $Comp
-L LED D?
+L LED D7
 U 1 1 53D64260
 P 1900 4200
-F 0 "D?" H 1900 4300 50  0000 C CNN
+F 0 "D7" H 1900 4300 50  0000 C CNN
 F 1 "LED" H 1900 4100 50  0000 C CNN
 F 2 "" H 1900 4200 60  0000 C CNN
@@
 $EndComp
 $Comp
-L LED D?
+L LED D8
 U 1 1 53D6426C
 P 1900 4500
-F 0 "D?" H 1900 4600 50  0000 C CNN
+F 0 "D8" H 1900 4600 50  0000 C CNN
 F 1 "LED" H 1900 4400 50  0000 C CNN
 F 2 "" H 1900 4500 60  0000 C CNN
@@
 $EndComp
 $Comp
-L LED D?
+L LED D9
 U 1 1 53D64272
 P 1900 4800
-F 0 "D?" H 1900 4900 50  0000 C CNN
+F 0 "D9" H 1900 4900 50  0000 C CNN
 F 1 "LED" H 1900 4700 50  0000 C CNN
 F 2 "" H 1900 4800 60  0000 C CNN
@@
 $EndComp
 $Comp
-L LED D?
+L LED D10
 U 1 1 53D64278
 P 1900 5100
-F 0 "D?" H 1900 5200 50  0000 C CNN
+F 0 "D10" H 1900 5200 50  0000 C CNN
 F 1 "LED" H 1900 5000 50  0000 C CNN
 F 2 "" H 1900 5100 60  0000 C CNN
@@
 $EndComp
 $Comp
-L BATTERY BT?
+L BATTERY BT1
 U 1 1 53D64296
 P 3050 900
-F 0 "BT?" H 3050 1100 50  0000 C CNN
+F 0 "BT1" H 3050 1100 50  0000 C CNN
 F 1 "BATTERY" H 3050 710 50  0000 C CNN
 F 2 "" H 3050 900 60  0000 C CNN
@@
 $EndComp
 $Comp
-L GND #PWR?
+L GND #PWR29
 U 1 1 53D642A5
 P 3350 1000
-F 0 "#PWR?" H 3350 1000 30  0001 C CNN
+F 0 "#PWR29" H 3350 1000 30  0001 C CNN
 F 1 "GND" H 3350 930 30  0001 C CNN
 F 2 "" H 3350 1000 60  0000 C CNN
@@
 	1700 5100 1500 5100
 $Comp
-L SPST SW?
+L SPST SW6
 U 1 1 53D643ED
 P 2150 900
-F 0 "SW?" H 2150 1000 70  0000 C CNN
+F 0 "SW6" H 2150 1000 70  0000 C CNN
 F 1 "SPST" H 2150 800 70  0000 C CNN
 F 2 "" H 2150 900 60  0000 C CNN
@@
 	1500 900  1650 900
 $Comp
-L GND #PWR?
+L GND #PWR30
 U 1 1 53D64527
 P 3550 2100
-F 0 "#PWR?" H 3550 2100 30  0001 C CNN
+F 0 "#PWR30" H 3550 2100 30  0001 C CNN
 F 1 "GND" H 3550 2030 30  0001 C CNN
 F 2 "" H 3550 2100 60  0000 C CNN
@@
 	4050 2500 4050 3150
 $Comp
-L GND #PWR?
+L GND #PWR31
 U 1 1 53D64679
 P 4050 3150
-F 0 "#PWR?" H 4050 3150 30  0001 C CNN
+F 0 "#PWR31" H 4050 3150 30  0001 C CNN
 F 1 "GND" H 4050 3080 30  0001 C CNN
 F 2 "" H 4050 3150 60  0000 C CNN
@@
 	3450 2950 3350 2950
 $Comp
-L SW_PUSH SW?
+L SW_PUSH SW2
 U 1 1 53D647DD
 P 1950 1750
-F 0 "SW?" H 2100 1860 50  0000 C CNN
+F 0 "SW2" H 2100 1860 50  0000 C CNN
 F 1 "SW_PUSH" H 1950 1670 50  0000 C CNN
 F 2 "" H 1950 1750 60  0000 C CNN
@@
 $EndComp
 $Comp
-L SW_PUSH SW?
+L SW_PUSH SW3
 U 1 1 53D647EA
 P 1950 2100
-F 0 "SW?" H 2100 2210 50  0000 C CNN
+F 0 "SW3" H 2100 2210 50  0000 C CNN
 F 1 "SW_PUSH" H 1950 2020 50  0000 C CNN
 F 2 "" H 1950 2100 60  0000 C CNN
@@
 $EndComp
 $Comp
-L SW_PUSH SW?
+L SW_PUSH SW4
 U 1 1 53D647F0
 P 1950 2500
-F 0 "SW?" H 2100 2610 50  0000 C CNN
+F 0 "SW4" H 2100 2610 50  0000 C CNN
 F 1 "SW_PUSH" H 1950 2420 50  0000 C CNN
 F 2 "" H 1950 2500 60  0000 C CNN
@@
 $EndComp
 $Comp
-L SW_PUSH SW?
+L SW_PUSH SW5
 U 1 1 53D647F6
 P 1950 2850
-F 0 "SW?" H 2100 2960 50  0000 C CNN
+F 0 "SW5" H 2100 2960 50  0000 C CNN
 F 1 "SW_PUSH" H 1950 2770 50  0000 C CNN
 F 2 "" H 1950 2850 60  0000 C CNN
@@
 	1500 2850 1650 2850
 $Comp
-L GND #PWR?
+L GND #PWR27
 U 1 1 53D6A2BE
 P 1650 1200
-F 0 "#PWR?" H 1650 1200 30  0001 C CNN
+F 0 "#PWR27" H 1650 1200 30  0001 C CNN
 F 1 "GND" H 1650 1130 30  0001 C CNN
 F 2 "" H 1650 1200 60  0000 C CNN
@@
 	2100 3600 2100 5100
 $Comp
-L R R?
+L R R8
 U 1 1 53D77D36
 P 2450 3300
-F 0 "R?" V 2530 3300 50  0000 C CNN
+F 0 "R8" V 2530 3300 50  0000 C CNN
 F 1 "330" V 2450 3300 50  0000 C CNN
 F 2 "" H 2450 3300 60  0000 C CNN
@@
 	2450 3600 2450 3550
 $Comp
-L GND #PWR?
+L GND #PWR28
 U 1 1 53D7DE63
 P 2100 1400
-F 0 "#PWR?" H 2100 1400 30  0001 C CNN
+F 0 "#PWR28" H 2100 1400 30  0001 C CNN
 F 1 "GND" H 2100 1330 30  0001 C CNN
 F 2 "" H 2100 1400 60  0000 C CNN

Commit message: Modified some code on "frum" and "microdrill"
Parts:
- renumbered D5 to D3, D6 to D4, D7 to D5, D8 to D6, D9 to D7, D10 to D8, R8 to R5, SW2 to SW1, SW3 to SW2, SW4 to SW3, SW5 to SW4, SW6 to SW5, X1 to X2, X2 to X3
Connections:
- no-connect marks 2 -> 0
Changed lines of the file:
@@
 Sheet 2 3
 Title ""
-Date "20 sep 2014"
+Date "13 oct 2014"
 Rev ""
 Comp ""
@@
 $EndComp
 $Comp
-L CRYSTAL X2
+L CRYSTAL X3
 U 1 1 53D64225
 P 3750 2950
-F 0 "X2" H 3750 3100 60  0000 C CNN
+F 0 "X3" H 3750 3100 60  0000 C CNN
 F 1 "CRYSTAL" H 3750 2800 60  0000 C CNN
 F 2 "" H 3750 2950 60  0000 C CNN
@@
 $EndComp
 $Comp
-L CRYSTAL X1
+L CRYSTAL X2
 U 1 1 53D64234
 P 3750 2500
-F 0 "X1" H 3750 2650 60  0000 C CNN
+F 0 "X2" H 3750 2650 60  0000 C CNN
 F 1 "CRYSTAL" H 3750 2350 60  0000 C CNN
 F 2 "" H 3750 2500 60  0000 C CNN
@@
 $EndComp
 $Comp
-L LED D5
+L LED D3
 U 1 1 53D6424D
 P 1900 3600
-F 0 "D5" H 1900 3700 50  0000 C CNN
+F 0 "D3" H 1900 3700 50  0000 C CNN
 F 1 "LED" H 1900 3500 50  0000 C CNN
 F 2 "" H 1900 3600 60  0000 C CNN
@@
 $EndComp
 $Comp
-L LED D6
+L LED D4
 U 1 1 53D6425A
 P 1900 3900
-F 0 "D6" H 1900 4000 50  0000 C CNN
+F 0 "D4" H 1900 4000 50  0000 C CNN
 F 1 "LED" H 1900 3800 50  0000 C CNN
 F 2 "" H 1900 3900 60  0000 C CNN
@@
 $EndComp
 $Comp
-L LED D7
+L LED D5
 U 1 1 53D64260
 P 1900 4200
-F 0 "D7" H 1900 4300 50  0000 C CNN
+F 0 "D5" H 1900 4300 50  0000 C CNN
 F 1 "LED" H 1900 4100 50  0000 C CNN
 F 2 "" H 1900 4200 60  0000 C CNN
@@
 $EndComp
 $Comp
-L LED D8
+L LED D6
 U 1 1 53D6426C
 P 1900 4500
-F 0 "D8" H 1900 4600 50  0000 C CNN
+F 0 "D6" H 1900 4600 50  0000 C CNN
 F 1 "LED" H 1900 4400 50  0000 C CNN
 F 2 "" H 1900 4500 60  0000 C CNN
@@
 $EndComp
 $Comp
-L LED D9
+L LED D7
 U 1 1 53D64272
 P 1900 4800
-F 0 "D9" H 1900 4900 50  0000 C CNN
+F 0 "D7" H 1900 4900 50  0000 C CNN
 F 1 "LED" H 1900 4700 50  0000 C CNN
 F 2 "" H 1900 4800 60  0000 C CNN
@@
 $EndComp
 $Comp
-L LED D10
+L LED D8
 U 1 1 53D64278
 P 1900 5100
-F 0 "D10" H 1900 5200 50  0000 C CNN
+F 0 "D8" H 1900 5200 50  0000 C CNN
 F 1 "LED" H 1900 5000 50  0000 C CNN
 F 2 "" H 1900 5100 60  0000 C CNN
@@
 $EndComp
 $Comp
-L GND #PWR29
+L GND #PWR023
 U 1 1 53D642A5
 P 3350 1000
-F 0 "#PWR29" H 3350 1000 30  0001 C CNN
+F 0 "#PWR023" H 3350 1000 30  0001 C CNN
 F 1 "GND" H 3350 930 30  0001 C CNN
 F 2 "" H 3350 1000 60  0000 C CNN
@@
 	1700 5100 1500 5100
 $Comp
-L SPST SW6
+L SPST SW5
 U 1 1 53D643ED
 P 2150 900
-F 0 "SW6" H 2150 1000 70  0000 C CNN
+F 0 "SW5" H 2150 1000 70  0000 C CNN
 F 1 "SPST" H 2150 800 70  0000 C CNN
 F 2 "" H 2150 900 60  0000 C CNN
@@
 	1500 900  1650 900
 $Comp
-L GND #PWR30
+L GND #PWR024
 U 1 1 53D64527
 P 3550 2100
-F 0 "#PWR30" H 3550 2100 30  0001 C CNN
+F 0 "#PWR024" H 3550 2100 30  0001 C CNN
 F 1 "GND" H 3550 2030 30  0001 C CNN
 F 2 "" H 3550 2100 60  0000 C CNN
@@
 	4050 2500 4050 3150
 $Comp
-L GND #PWR31
+L GND #PWR025
 U 1 1 53D64679
 P 4050 3150
-F 0 "#PWR31" H 4050 3150 30  0001 C CNN
+F 0 "#PWR025" H 4050 3150 30  0001 C CNN
 F 1 "GND" H 4050 3080 30  0001 C CNN
 F 2 "" H 4050 3150 60  0000 C CNN
@@
 	3450 2950 3350 2950
 $Comp
-L SW_PUSH SW2
+L SW_PUSH SW1
 U 1 1 53D647DD
 P 1950 1750
-F 0 "SW2" H 2100 1860 50  0000 C CNN
+F 0 "SW1" H 2100 1860 50  0000 C CNN
 F 1 "SW_PUSH" H 1950 1670 50  0000 C CNN
 F 2 "" H 1950 1750 60  0000 C CNN
@@
 $EndComp
 $Comp
-L SW_PUSH SW3
+L SW_PUSH SW2
 U 1 1 53D647EA
 P 1950 2100
-F 0 "SW3" H 2100 2210 50  0000 C CNN
+F 0 "SW2" H 2100 2210 50  0000 C CNN
 F 1 "SW_PUSH" H 1950 2020 50  0000 C CNN
 F 2 "" H 1950 2100 60  0000 C CNN
@@
 $EndComp
 $Comp
-L SW_PUSH SW4
+L SW_PUSH SW3
 U 1 1 53D647F0
 P 1950 2500
-F 0 "SW4" H 2100 2610 50  0000 C CNN
+F 0 "SW3" H 2100 2610 50  0000 C CNN
 F 1 "SW_PUSH" H 1950 2420 50  0000 C CNN
 F 2 "" H 1950 2500 60  0000 C CNN
@@
 $EndComp
 $Comp
-L SW_PUSH SW5
+L SW_PUSH SW4
 U 1 1 53D647F6
 P 1950 2850
-F 0 "SW5" H 2100 2960 50  0000 C CNN
+F 0 "SW4" H 2100 2960 50  0000 C CNN
 F 1 "SW_PUSH" H 1950 2770 50  0000 C CNN
 F 2 "" H 1950 2850 60  0000 C CNN
@@
 	1500 2850 1650 2850
 $Comp
-L GND #PWR27
+L GND #PWR026
 U 1 1 53D6A2BE
 P 1650 1200
-F 0 "#PWR27" H 1650 1200 30  0001 C CNN
+F 0 "#PWR026" H 1650 1200 30  0001 C CNN
 F 1 "GND" H 1650 1130 30  0001 C CNN
 F 2 "" H 1650 1200 60  0000 C CNN
@@
 	2100 3600 2100 5100
 $Comp
-L R R8
+L R R5
 U 1 1 53D77D36
 P 2450 3300
-F 0 "R8" V 2530 3300 50  0000 C CNN
+F 0 "R5" V 2530 3300 50  0000 C CNN
 F 1 "330" V 2450 3300 50  0000 C CNN
 F 2 "" H 2450 3300 60  0000 C CNN
@@
 	2450 1150 1800 1150
 Connection ~ 1800 1150
-NoConn ~ 1950 1300
-NoConn ~ 2100 1300
 Text Notes 1050 1450 0    60   ~ 0
 Break here\nand connect to GROUND!
@@
 	2450 3600 2450 3550
 $Comp
-L GND #PWR28
+L GND #PWR027
 U 1 1 53D7DE63
 P 2100 1400
-F 0 "#PWR28" H 2100 1400 30  0001 C CNN
+F 0 "#PWR027" H 2100 1400 30  0001 C CNN
 F 1 "GND" H 2100 1330 30  0001 C CNN
 F 2 "" H 2100 1400 60  0000 C CNN
@@
 	2100 1350 2250 1350
 Connection ~ 2250 1350
+Wire Notes Line
+	1900 1250 2150 1250
+$Comp
+L PWR_FLAG #FLG028
+U 1 1 5426B7EA
+P 1550 1150
+F 0 "#FLG028" H 1550 1245 30  0001 C CNN
+F 1 "PWR_FLAG" H 1550 1330 30  0000 C CNN
+F 2 "" H 1550 1150 60  0000 C CNN
+F 3 "" H 1550 1150 60  0000 C CNN
+	1    1550 1150
+	1    0    0    -1
+$EndComp
+Connection ~ 1550 1150
 $EndSCHEMATC
