File: DRUM/schematics/Player.sch (KiCad schematic (older format))
At the start: 6 parts

Commit message: modified DRUM schematics
Parts:
- removed SW? (x5): SW_PUSH, symbol SW_PUSH
- added P5, P6, P7, P8, P9: CONN_2, symbol CONN_2
- gave numbers to parts that had none: 1
Connections:
- net BTN0a: now also P5.1 (P1)
- net BTN0b: now also P5.2 (PM)
- net BTN1a: now also P6.1 (P1)
- net BTN1b: now also P6.2 (PM)
- net BTN2a: now also P7.1 (P1)
- net BTN2b: now also P7.2 (PM)
- net BTN3a: now also P8.1 (P1)
- net BTN3b: now also P8.2 (PM)
- net BTN4a: now also P9.1 (P1)
- net BTN4b: now also P9.2 (PM)
Other:
- note added: "Buttons' contacts mark:\n"a" - inner circle;\n"b" - outern ring"
Changed lines of the file:
@@
 LIBS:tda2822
 LIBS:CD74HC154
+LIBS:transistors_gaui
 LIBS:drum-cache
 EELAYER 27 0
@@
 Sheet 3 3
 Title ""
-Date "28 jul 2014"
+Date "20 sep 2014"
 Rev ""
 Comp ""
@@
 $EndDescr
 $Comp
-L SW_PUSH SW?
-U 1 1 53D66E36
-P 1700 2050
-F 0 "SW?" H 1850 2160 50  0000 C CNN
-F 1 "SW_PUSH" H 1700 1970 50  0000 C CNN
-F 2 "" H 1700 2050 60  0000 C CNN
-F 3 "" H 1700 2050 60  0000 C CNN
-	1    1700 2050
-	1    0    0    -1
-$EndComp
-$Comp
-L BATTERY BT?
+L BATTERY BT2
 U 1 1 53D66E57
 P 1450 4300
-F 0 "BT?" H 1450 4500 50  0000 C CNN
+F 0 "BT2" H 1450 4500 50  0000 C CNN
 F 1 "BATTERY" H 1450 4110 50  0000 C CNN
 F 2 "" H 1450 4300 60  0000 C CNN
@@
 Wire Wire Line
 	1400 2050 1200 2050
-Wire Wire Line
-	2000 2050 2000 1850
-Wire Wire Line
-	2000 1850 1200 1850
-$Comp
-L SW_PUSH SW?
-U 1 1 53D66E75
-P 1700 2450
-F 0 "SW?" H 1850 2560 50  0000 C CNN
-F 1 "SW_PUSH" H 1700 2370 50  0000 C CNN
-F 2 "" H 1700 2450 60  0000 C CNN
-F 3 "" H 1700 2450 60  0000 C CNN
-	1    1700 2450
-	1    0    0    -1
-$EndComp
-Wire Wire Line
-	1400 2450 1200 2450
-Wire Wire Line
-	2000 2450 2000 2250
-Wire Wire Line
-	2000 2250 1200 2250
-$Comp
-L SW_PUSH SW?
-U 1 1 53D66E80
-P 1700 2850
-F 0 "SW?" H 1850 2960 50  0000 C CNN
-F 1 "SW_PUSH" H 1700 2770 50  0000 C CNN
-F 2 "" H 1700 2850 60  0000 C CNN
-F 3 "" H 1700 2850 60  0000 C CNN
-	1    1700 2850
-	1    0    0    -1
-$EndComp
-Wire Wire Line
-	1400 2850 1200 2850
-Wire Wire Line
-	2000 2850 2000 2650
-Wire Wire Line
-	2000 2650 1200 2650
-$Comp
-L SW_PUSH SW?
-U 1 1 53D66E8B
-P 1700 3250
-F 0 "SW?" H 1850 3360 50  0000 C CNN
-F 1 "SW_PUSH" H 1700 3170 50  0000 C CNN
-F 2 "" H 1700 3250 60  0000 C CNN
-F 3 "" H 1700 3250 60  0000 C CNN
-	1    1700 3250
-	1    0    0    -1
-$EndComp
-Wire Wire Line
-	1400 3250 1200 3250
-Wire Wire Line
-	2000 3250 2000 3050
-Wire Wire Line
-	2000 3050 1200 3050
-$Comp
-L SW_PUSH SW?
-U 1 1 53D66E9C
-P 1700 3650
-F 0 "SW?" H 1850 3760 50  0000 C CNN
-F 1 "SW_PUSH" H 1700 3570 50  0000 C CNN
-F 2 "" H 1700 3650 60  0000 C CNN
-F 3 "" H 1700 3650 60  0000 C CNN
-	1    1700 3650
-	1    0    0    -1
-$EndComp
-Wire Wire Line
-	1400 3650 1200 3650
-Wire Wire Line
-	2000 3650 2000 3450
-Wire Wire Line
-	2000 3450 1200 3450
 Text HLabel 1200 1850 0    60   Input ~ 0
 BTN0a
@@
 Connection ~ 1450 4600
 $Comp
-L PWR_FLAG #FLG?
+L PWR_FLAG #FLG1
 U 1 1 53D67208
 P 1300 4900
-F 0 "#FLG?" H 1300 4995 30  0001 C CNN
+F 0 "#FLG1" H 1300 4995 30  0001 C CNN
 F 1 "PWR_FLAG" H 1300 5080 30  0000 C CNN
 F 2 "" H 1300 4900 60  0000 C CNN
@@
 $EndComp
 $Comp
-L PWR_FLAG #FLG?
+L PWR_FLAG #FLG2
 U 1 1 53D67215
 P 1600 5100
-F 0 "#FLG?" H 1600 5195 30  0001 C CNN
+F 0 "#FLG2" H 1600 5195 30  0001 C CNN
 F 1 "PWR_FLAG" H 1600 5280 30  0000 C CNN
 F 2 "" H 1600 5100 60  0000 C CNN
@@
 Wire Wire Line
 	1200 4900 1300 4900
+$Comp
+L CONN_2 P5
+U 1 1 541D2C34
+P 1750 1950
+F 0 "P5" V 1700 1950 40  0000 C CNN
+F 1 "CONN_2" V 1800 1950 40  0000 C CNN
+F 2 "" H 1750 1950 60  0000 C CNN
+F 3 "" H 1750 1950 60  0000 C CNN
+	1    1750 1950
+	1    0    0    -1
+$EndComp
+Wire Wire Line
+	1200 1850 1400 1850
+Wire Wire Line
+	1400 2450 1200 2450
+$Comp
+L CONN_2 P6
+U 1 1 541D2C57
+P 1750 2350
+F 0 "P6" V 1700 2350 40  0000 C CNN
+F 1 "CONN_2" V 1800 2350 40  0000 C CNN
+F 2 "" H 1750 2350 60  0000 C CNN
+F 3 "" H 1750 2350 60  0000 C CNN
+	1    1750 2350
+	1    0    0    -1
+$EndComp
+Wire Wire Line
+	1200 2250 1400 2250
+Wire Wire Line
+	1400 2850 1200 2850
+$Comp
+L CONN_2 P7
+U 1 1 541D2C5F
+P 1750 2750
+F 0 "P7" V 1700 2750 40  0000 C CNN
+F 1 "CONN_2" V 1800 2750 40  0000 C CNN
+F 2 "" H 1750 2750 60  0000 C CNN
+F 3 "" H 1750 2750 60  0000 C CNN
+	1    1750 2750
+	1    0    0    -1
+$EndComp
+Wire Wire Line
+	1200 2650 1400 2650
+Wire Wire Line
+	1400 3250 1200 3250
+$Comp
+L CONN_2 P8
+U 1 1 541D2C67
+P 1750 3150
+F 0 "P8" V 1700 3150 40  0000 C CNN
+F 1 "CONN_2" V 1800 3150 40  0000 C CNN
+F 2 "" H 1750 3150 60  0000 C CNN
+F 3 "" H 1750 3150 60  0000 C CNN
+	1    1750 3150
+	1    0    0    -1
+$EndComp
+Wire Wire Line
+	1200 3050 1400 3050
+Wire Wire Line
+	1400 3650 1200 3650
+$Comp
+L CONN_2 P9
+U 1 1 541D2C6F
+P 1750 3550
+F 0 "P9" V 1700 3550 40  0000 C CNN
+F 1 "CONN_2" V 1800 3550 40  0000 C CNN
+F 2 "" H 1750 3550 60  0000 C CNN
+F 3 "" H 1750 3550 60  0000 C CNN
+	1    1750 3550
+	1    0    0    -1
+$EndComp
+Wire Wire Line
+	1200 3450 1400 3450
+Text Notes 900  1500 0    60   ~ 0
+Buttons' contacts mark:\n"a" - inner circle;\n"b" - outern ring
 $EndSCHEMATC

Commit message: Modified some code on "frum" and "microdrill"
Parts:
- renumbered P5 to P2, P6 to P3, P7 to P4, P8 to P5, P9 to P6
Connections:
- net BAT- renamed SND_gnd
Changed lines of the file:
@@
 Sheet 3 3
 Title ""
-Date "20 sep 2014"
+Date "13 oct 2014"
 Rev ""
 Comp ""
@@
 Text HLabel 1200 4000 0    60   Input ~ 0
 BAT+
-Text HLabel 1200 4600 0    60   Input ~ 0
-BAT-
-Wire Wire Line
-	1200 4600 1450 4600
 Wire Wire Line
 	1200 4000 1450 4000
@@
 Wire Wire Line
 	1450 5300 1450 4600
-Connection ~ 1450 4600
 $Comp
-L PWR_FLAG #FLG1
+L PWR_FLAG #FLG029
 U 1 1 53D67208
 P 1300 4900
-F 0 "#FLG1" H 1300 4995 30  0001 C CNN
+F 0 "#FLG029" H 1300 4995 30  0001 C CNN
 F 1 "PWR_FLAG" H 1300 5080 30  0000 C CNN
 F 2 "" H 1300 4900 60  0000 C CNN
@@
 $EndComp
 $Comp
-L PWR_FLAG #FLG2
+L PWR_FLAG #FLG030
 U 1 1 53D67215
 P 1600 5100
-F 0 "#FLG2" H 1600 5195 30  0001 C CNN
+F 0 "#FLG030" H 1600 5195 30  0001 C CNN
 F 1 "PWR_FLAG" H 1600 5280 30  0000 C CNN
 F 2 "" H 1600 5100 60  0000 C CNN
@@
 	1200 4900 1300 4900
 $Comp
-L CONN_2 P5
+L CONN_2 P2
 U 1 1 541D2C34
 P 1750 1950
-F 0 "P5" V 1700 1950 40  0000 C CNN
+F 0 "P2" V 1700 1950 40  0000 C CNN
 F 1 "CONN_2" V 1800 1950 40  0000 C CNN
 F 2 "" H 1750 1950 60  0000 C CNN
@@
 	1400 2450 1200 2450
 $Comp
-L CONN_2 P6
+L CONN_2 P3
 U 1 1 541D2C57
 P 1750 2350
-F 0 "P6" V 1700 2350 40  0000 C CNN
+F 0 "P3" V 1700 2350 40  0000 C CNN
 F 1 "CONN_2" V 1800 2350 40  0000 C CNN
 F 2 "" H 1750 2350 60  0000 C CNN
@@
 	1400 2850 1200 2850
 $Comp
-L CONN_2 P7
+L CONN_2 P4
 U 1 1 541D2C5F
 P 1750 2750
-F 0 "P7" V 1700 2750 40  0000 C CNN
+F 0 "P4" V 1700 2750 40  0000 C CNN
 F 1 "CONN_2" V 1800 2750 40  0000 C CNN
 F 2 "" H 1750 2750 60  0000 C CNN
@@
 	1400 3250 1200 3250
 $Comp
-L CONN_2 P8
+L CONN_2 P5
 U 1 1 541D2C67
 P 1750 3150
-F 0 "P8" V 1700 3150 40  0000 C CNN
+F 0 "P5" V 1700 3150 40  0000 C CNN
 F 1 "CONN_2" V 1800 3150 40  0000 C CNN
 F 2 "" H 1750 3150 60  0000 C CNN
@@
 	1400 3650 1200 3650
 $Comp
-L CONN_2 P9
+L CONN_2 P6
 U 1 1 541D2C6F
 P 1750 3550
-F 0 "P9" V 1700 3550 40  0000 C CNN
+F 0 "P6" V 1700 3550 40  0000 C CNN
 F 1 "CONN_2" V 1800 3550 40  0000 C CNN
 F 2 "" H 1750 3550 60  0000 C CNN
