File: DRUM/schematics/drum.sch (KiCad schematic (older format))
At the start: 27 parts, among them P1 CONN_14, P2 CONN_4, P3 CONN_14, P4 CONN_5, SW1 SW_PUSH, U1 STM8S105K4T6C

Commit message: Fixed error in ULN stepper management + added simple work with bipolar steppers by two L9110s H-bridge drivers
Connections:
- wire segments 87 -> 86
Other:
- note added: "LEDs off"
Changed lines of the file:
@@
 Sheet 1 3
 Title ""
-Date "28 jul 2014"
+Date "30 jul 2014"
 Rev ""
 Comp ""
@@
 NoConn ~ 12800 3400
 NoConn ~ 12800 3300
-Wire Wire Line
-	12800 3100 12800 3200
 $Comp
 L GND #PWR?
@@
 Wire Wire Line
 	13000 3200 12800 3200
-Connection ~ 12800 3200
 Text Notes 2050 3450 0    60   ~ 0
 LEDs address 3\n2\n1\n0
-Text Notes 2150 3250 0    60   ~ 0
+Text Notes 2650 3050 0    60   ~ 0
 DRUM0\nDRUM1
 Text Label 12800 3000 0    60   ~ 0
@@
 Text Label 12800 2700 0    60   ~ 0
 PB0
-Text Label 10900 4100 0    60   ~ 0
+Text Label 12800 3100 0    60   ~ 0
 PB4
 Text Label 10900 4250 0    60   ~ 0
@@
 Wire Wire Line
 	10800 4100 10900 4100
+Text Label 10900 4100 0    60   ~ 0
+PF4
+Text Notes 2400 3350 0    60   ~ 0
+LEDs off
 $EndSCHEMATC

Commit message: modified DRUM schematics
Parts:
- removed C? (x2): 100u, symbol C
- removed C?: 0.1u, symbol C
- removed R?: 4R7, symbol R
- removed R? (x2): 10k, symbol R
- added D3, D4: BZX55C3V6, symbol ZENERSMALL
- added Q1, Q2, Q3, Q4, Q5, Q6: 2N7002, transistors_gaui-SOT23, symbol 2N7002
- added R4, R5, R7: 10k, SM0603, symbol R
- added R6: 3.3k, SM0603, symbol R
- gave numbers to parts that had none: 6
Connections:
- net labels added: Next_circle, Next_ring, Play_circle, Play_ring, Prev_circle, Prev_ring, Vol+_circle, Vol+_ring, Vol-_circle, Vol-_ring
- wire segments 86 -> 121
Other:
- note added: "Player buttons\ncontrol: PD0..PD4"
- moved on the sheet: C4, C5, R3

Commit message: Modified some code on "frum" and "microdrill"
Parts:
- removed C1: 1u, symbol C
- removed C2, C3: 104, symbol C
- removed C6, C7: 100u, symbol C
- removed D1, D2: LED, symbol LED
- removed P1, P3: CONN_14, symbol CONN_14
- removed P2: CONN_4, symbol CONN_4
- removed R1, R2: 1k, symbol R
- removed R3: 10k, symbol R
- removed SW1: SW_PUSH, symbol SW_PUSH
- removed U1: STM8S105K4T6C, ~, symbol STM8S105K4T6C
- added C3, C4: 100u, ~, symbol CP1
- added D9: DIODESCH, ~, symbol DIODESCH
- added P10, P11, P12, P13, P15, P16, P18, P19, P20, P21, P22, P23, P24, P25, P26, P27, P28, P29, P8, P9: CONN_1, symbol CONN_1
- added P7: CONN_10, symbol CONN_10
- added R6: 100k, SM0603, symbol R
- added X1: STM8S105BOARD, devboard_pins-9-14, symbol STM8S105BOARD
- DA1: footprint DIP-4__300 -> DIP-8__300
- renumbered C4 to C1, C5 to C2, D3 to D1, D4 to D2, P4 to P1, R4 to R1, R5 to R2, R6 to R3, R7 to R4
Connections:
- net labels added: Audio_in, LED0, LED1, LED2, LED3, LED4, LED5
- net labels removed: +3.3V
- wire segments 121 -> 97
- no-connect marks 13 -> 16
Other:
- note added: "Acc. Voltage"
- note added: "Bat. Voltage"
- note added: "CONNECTORS"
- note added: "LEDs address 1\n0"
- note added: "LEDs address 2"
- note added: "Mount on wires"
- note added: "Ref. Voltage"
- note added: "Solder C1-C2\non wires"
- note added: "Solder zeners directly on piezo"
- note removed: "LEDs address 3\n2\n1\n0"
- note removed: "STM8 board"

Commit message: started voltmeter hacking
Parts:
- removed D1, D2: BZX55C3V6, symbol ZENERSMALL
- removed X1: STM8S105BOARD, devboard_pins-9-14, symbol STM8S105BOARD
- added D1, D2: BZX55C3V6, symbol ZENERsmall
- added X1: stm8s105board, devboard_pins-9-14, symbol stm8s105board
Changed lines of the file:
@@
 LIBS:tda2822
 LIBS:CD74HC154
-LIBS:transistors_gaui
 LIBS:drum-cache
-EELAYER 27 0
+EELAYER 24 0
 EELAYER END
 $Descr A3 16535 11693
@@
 Play_circle
 $Comp
-L ZENERSMALL D1
-U 1 1 541D94C6
-P 11100 4350
-F 0 "D1" H 11100 4450 40  0000 C CNN
-F 1 "BZX55C3V6" H 11100 4250 30  0000 C CNN
-F 2 "" H 11100 4350 60  0000 C CNN
-F 3 "" H 11100 4350 60  0000 C CNN
-	1    11100 4350
-	0    -1   -1   0
-$EndComp
-$Comp
-L ZENERSMALL D2
-U 1 1 541D9B34
-P 11400 4350
-F 0 "D2" H 11400 4450 40  0000 C CNN
-F 1 "BZX55C3V6" H 11400 4250 30  0000 C CNN
-F 2 "" H 11400 4350 60  0000 C CNN
-F 3 "" H 11400 4350 60  0000 C CNN
-	1    11400 4350
-	0    -1   -1   0
-$EndComp
-$Comp
 L GND #PWR013
 U 1 1 541D9D40
@@
 Wire Wire Line
 	6500 7500 6600 7500
-$Comp
-L STM8S105BOARD X1
-U 1 1 5425C192
-P 3900 2500
-F 0 "X1" H 3900 3550 60  0000 C CNN
-F 1 "STM8S105BOARD" H 3900 1850 60  0000 C CNN
-F 2 "devboard_pins-9-14" H 3900 2500 60  0001 C CNN
-F 3 "~" H 3900 2500 60  0000 C CNN
-	1    3900 2500
-	1    0    0    -1
-$EndComp
 Wire Wire Line
 	2500 1650 2500 1600
@@
 	1    0    0    -1
 $EndComp
+$Comp
+L stm8s105board X1
+U 1 1 54A06126
+P 3900 2500
+F 0 "X1" H 3900 3550 60  0000 C CNN
+F 1 "stm8s105board" H 3900 1850 60  0000 C CNN
+F 2 "devboard_pins-9-14" H 3900 2500 60  0001 C CNN
+F 3 "" H 3900 2500 60  0000 C CNN
+	1    3900 2500
+	1    0    0    -1
+$EndComp
+$Comp
+L ZENERsmall D1
+U 1 1 54A0D38A
+P 11100 4350
+F 0 "D1" H 11100 4450 40  0000 C CNN
+F 1 "BZX55C3V6" H 11100 4250 30  0000 C CNN
+F 2 "" H 11100 4350 60  0000 C CNN
+F 3 "" H 11100 4350 60  0000 C CNN
+	1    11100 4350
+	0    -1   -1   0
+$EndComp
+$Comp
+L ZENERsmall D2
+U 1 1 54A0DB5F
+P 11400 4350
+F 0 "D2" H 11400 4450 40  0000 C CNN
+F 1 "BZX55C3V6" H 11400 4250 30  0000 C CNN
+F 2 "" H 11400 4350 60  0000 C CNN
+F 3 "" H 11400 4350 60  0000 C CNN
+	1    11400 4350
+	0    -1   -1   0
+$EndComp
 $EndSCHEMATC
