File: 220controlled_socket/kicad/socket.kicad_pcb (KiCad board)
At the start: 2 copper layers, 87 x 71 mm, 85 parts, among them J1 DB9_Female, J2 USB_B, J3 5Vext, J4 SWIM, J5 DB15_Male, J6 Power, J7 Power, K1 SRD-05VDC, K2 SRD-05VDC, Q1 2N7002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

Commit message: partially worked microdrill
Parts:
- added C14: 0.01 600V, Capacitor_THT:C_Disc_D6.0mm_W2.5mm_P5.00mm, F.Cu at (121.9, 49.5)
- added C15: 0.01 600V, Capacitor_THT:C_Disc_D6.0mm_W2.5mm_P5.00mm, F.Cu at (108.5, 80.5)
- added R34: 330 2W, Resistor_THT:R_Axial_Power_L20.0mm_W6.4mm_P25.40mm, B.Cu at (114.1, 49.5)
- added R35: 330 2W, Resistor_THT:R_Axial_Power_L20.0mm_W6.4mm_P25.40mm, B.Cu at (112.9, 90.6)
- R19, R21: footprint Resistor_THT:R_Axial_DIN0309_L9.0mm_D3.2mm_P12.70mm_Horizontal -> Resistor_SMD:R_1206_HandSoldering
- R20, R22: footprint Resistor_SMD:R_1206_3216Metric_Pad1.24x1.80mm_HandSolder -> Resistor_SMD:R_1206_HandSoldering
- moved R17 7.37 mm to (111.5, 51.5), turned to 90 degrees
- moved R21 3.64 mm to (103.0, 67.0)
- moved R19 2.67 mm to (95.0, 40.0)
Connections:
- J6 pad 2: GNDREF -> /NC1
- J7 pad 2: GNDREF -> /NC2
- K1 pad 4: (no net) -> /NC1
- K2 pad 4: (no net) -> /NC2
Routing:
- net GNDREF: track 46.8 -> 0.00 mm
- net /NC1: track 0.00 -> 31.9 mm
- net /NC2: track 0.00 -> 22.9 mm
- net Net-(C15-Pad1): track 44.5 -> 58.7 mm
- net Net-(D3-Pad2): track 44.2 -> 55.9 mm
- net Net-(R17-Pad1): track 2.63 -> 10.5 mm
- net Net-(C14-Pad1): track 10.5 -> 18.1 mm
- net VCC: track 256.8 -> 249.9 mm
- net Net-(C15-Pad2): track 0.00 -> 6.87 mm
- net Net-(D4-Pad3): track 19.9 -> 13.7 mm
- net Net-(D4-Pad2): track 39.5 -> 44.9 mm
- net Net-(D3-Pad1): track 32.4 -> 37.3 mm
- net Net-(D3-Pad3): track 12.9 -> 9.50 mm
- net GND: track 524.6 -> 527.8 mm
- net Net-(C14-Pad2): track 0.00 -> 2.75 mm
Other:
- board text added: "L1"
- board text added: "L2"
- board text added: "NC1"
- board text added: "NC2"
