File: 220controlled_socket/kicad/socket.sch (KiCad schematic (older format))
At the start: 67 parts, among them J1 DB9_Female, J2 USB_B, J3 5Vext, J4 SWIM, J5 DB15_Male, J6 Power, J7 Power, K1 SRD-05VDC, K2 SRD-05VDC, Q1 2N7002, Q2 2N7002, Q3 SI2300, Q4 SI2300, Q6 AO3407, Q8 2N7002, Q9 2N7002, U1 MAX3232, U10 ACS712, U2 CH340G, U3 STM8S003F3P, U5 PC817, U6 PC817, U7 PC817, U8 MOC3063M, U9 MOC3063M, Y1 12M

Commit message: 220v socket schematic is over
Parts:
- C12: footprint Capacitor_SMD:C_0805_2012Metric_Pad1.15x1.50mm_HandSolder -> Capacitor_SMD:C_0603_1608Metric_Pad0.84x1.00mm_HandSolder
- K1, K2: symbol SANYOU_SRD_Form_C -> G5LE-1
- R15, R17: value 100 -> 150
- R19, R21: footprint Resistor_SMD:R_1206_3216Metric_Pad1.24x1.80mm_HandSolder -> Resistor_THT:R_Axial_DIN0309_L9.0mm_D3.2mm_P12.70mm_Horizontal
- R24: footprint Resistor_SMD:R_0603_1608Metric_Pad0.84x1.00mm_HandSolder -> Resistor_SMD:R_0805_2012Metric_Pad1.15x1.50mm_HandSolder
- U3: symbol STM8S003F3P -> STM8S003F3P-RESCUE-socket
Connections:
- wire segments 178 -> 177
Other:
- moved on the sheet: C11, C12, C13, D6, Q1, Q2, R10, R3, R4, R5, R7, R8

Commit message: fix error in U5 connection on 220v socket
Parts:
- removed Q6: AO3407, Package_TO_SOT_SMD:SOT-23_Handsoldering, symbol Q_NMOS_GSD
- added Q6: AO3407, Package_TO_SOT_SMD:SOT-23_Handsoldering, symbol Q_PMOS_GSD
Connections:
- wire segments 177 -> 179
Changed lines of the file:
@@
 LIBS:ch34x
 LIBS:bt137
-LIBS:MCU_ST_STM8
-LIBS:Relay_SolidState
-LIBS:Device
-LIBS:Diode
-LIBS:Relay
-LIBS:Triac_Thyristor
-LIBS:Interface_UART
-LIBS:Power_Protection
-LIBS:Connector_Specialized
-LIBS:Connector_Generic
 LIBS:power
 LIBS:acs712
-LIBS:Isolator
+LIBS:transistors
 LIBS:socket-cache
 EELAYER 25 0
@@
 Text Label 4750 4400 2    60   ~ 0
 ~In0
-Text Label 4750 4800 2    60   ~ 0
+Text Label 4900 5000 2    60   ~ 0
 ~In1
 Text Label 3300 5800 2    60   ~ 0
@@
 	0    1    1    0
 $EndComp
-$Comp
-L Q_NMOS_GSD Q6
-U 1 1 5A7B0D05
-P 7100 3350
-F 0 "Q6" H 7300 3400 50  0000 L CNN
-F 1 "AO3407" H 7300 3300 50  0000 L CNN
-F 2 "Package_TO_SOT_SMD:SOT-23_Handsoldering" H 7300 3450 50  0001 C CNN
-F 3 "" H 7100 3350 50  0001 C CNN
-	1    7100 3350
-	1    0    0    1
-$EndComp
 Wire Wire Line
 	1900 2200 1900 2500
@@
 	9900 3900 9900 5000
 Wire Wire Line
-	10750 3950 10750 3750
+	10750 3750 10750 3950
 Wire Wire Line
 	10750 3750 10850 3750
@@
 	5000 4600 5000 5050
 Wire Wire Line
-	5000 5000 5100 5000
-Wire Wire Line
 	5000 4600 6100 4600
-Connection ~ 5000 5000
-Wire Wire Line
-	5100 4800 4750 4800
 Wire Wire Line
 	7650 5850 5800 5850
 Wire Wire Line
-	5800 5000 5700 5000
-Wire Wire Line
 	6050 5650 7650 5650
-Wire Wire Line
-	6050 4800 6050 5650
 Wire Wire Line
 	7650 5450 6100 5450
@@
 Wire Wire Line
 	7650 4650 7600 4650
-Wire Wire Line
-	7600 4650 7600 3150
 Wire Wire Line
 	7600 3150 7200 3150
@@
 	10900 3900 10750 3900
 Connection ~ 10750 3900
-Wire Wire Line
-	7650 4850 7200 4850
-Wire Wire Line
-	7200 4850 7200 3550
 NoConn ~ 7650 5050
 Wire Wire Line
-	7650 4950 6350 4950
-Wire Wire Line
-	6350 4950 6350 4050
+	6350 4950 7650 4950
+Wire Wire Line
+	6350 4050 6350 4950
 NoConn ~ 7650 5150
 $Comp
@@
 	5800 5850 5800 5300
 Wire Wire Line
-	5700 4800 6050 4800
-Wire Wire Line
 	6800 2050 6250 2050
 $Comp
@@
 	9200 1800 9200 1000
 Wire Wire Line
-	8850 2400 9050 2400
-Wire Wire Line
-	9050 2400 9050 1300
+	9050 2400 8850 2400
+Wire Wire Line
+	9050 1300 9050 2400
 Wire Wire Line
 	9900 5000 9700 5000
@@
 Wire Wire Line
 	10050 4400 10050 3600
+Wire Wire Line
+	4900 5000 5100 5000
+Wire Wire Line
+	5100 4800 5000 4800
+Connection ~ 5000 4800
+$Comp
+L Q_PMOS_GSD Q6
+U 1 1 5ACFAF39
+P 7100 3350
+F 0 "Q6" H 7300 3400 50  0000 L CNN
+F 1 "AO3407" H 7300 3300 50  0000 L CNN
+F 2 "Package_TO_SOT_SMD:SOT-23_Handsoldering" H 7300 3450 50  0001 C CNN
+F 3 "" H 7100 3350 50  0001 C CNN
+	1    7100 3350
+	1    0    0    1
+$EndComp
+Wire Wire Line
+	7200 4850 7200 3550
+Wire Wire Line
+	7650 4850 7200 4850
+Wire Wire Line
+	7600 4650 7600 3150
+Wire Wire Line
+	5800 5000 5800 4800
+Wire Wire Line
+	5800 4800 5700 4800
+Wire Wire Line
+	5700 5000 5700 4950
+Wire Wire Line
+	5700 4950 6050 4950
+Wire Wire Line
+	6050 4950 6050 5650
 $EndSCHEMATC

Commit message: fix bugs in 220v socket schematics
Parts:
- added Q5, Q7: 2N7002, Package_TO_SOT_SMD:SOT-23_Handsoldering, symbol Q_NMOS_GSD
- added R13, R25, R26, R27, R29, R30, R32, R33, R6: 47k, Resistor_SMD:R_0805_2012Metric_Pad1.15x1.50mm_HandSolder, symbol R
- added R28, R31: 330, Resistor_SMD:R_0603_1608Metric_Pad0.84x1.00mm_HandSolder, symbol R
Connections:
- wire segments 179 -> 200
Other:
- moved on the sheet: R12, R15, R17

Commit message: fix bug in max3232 & ch340 connection
Parts:
- removed R24: 510, Resistor_SMD:R_0805_2012Metric_Pad1.15x1.50mm_HandSolder, symbol R
- added D7, D8: SS14, Diode_SMD:D_SMA, symbol D
- R23: value 510 -> 4k7
Changed lines of the file:
@@
 Text Label 3850 2700 0    60   ~ 0
 Tx
-Text Label 4150 3400 0    60   ~ 0
+Text Label 4300 3100 0    60   ~ 0
 Rx
 $Comp
@@
 Text Label 2850 4650 2    60   ~ 0
 Tx
-Text Label 2750 3950 0    60   ~ 0
+Text Label 2700 4000 0    60   ~ 0
 Rx
 NoConn ~ 3750 4550
@@
 NKEY1
 $Comp
-L R R24
-U 1 1 5A7AA1DA
-P 4050 3250
-F 0 "R24" V 4130 3250 50  0000 C CNN
-F 1 "510" V 4050 3250 50  0000 C CNN
-F 2 "Resistor_SMD:R_0805_2012Metric_Pad1.15x1.50mm_HandSolder" V 3980 3250 50  0001 C CNN
-F 3 "" H 4050 3250 50  0001 C CNN
-	1    4050 3250
-	-1   0    0    1
-$EndComp
-$Comp
-L R R23
-U 1 1 5A7AB2E3
-P 2700 4150
-F 0 "R23" V 2780 4150 50  0000 C CNN
-F 1 "510" V 2700 4150 50  0000 C CNN
-F 2 "Resistor_SMD:R_0603_1608Metric_Pad0.84x1.00mm_HandSolder" V 2630 4150 50  0001 C CNN
-F 3 "" H 2700 4150 50  0001 C CNN
-	1    2700 4150
-	-1   0    0    1
-$EndComp
-$Comp
 L PWR_FLAG #FLG034
 U 1 1 5A7AD9A0
@@
 Connection ~ 9400 3950
 Wire Wire Line
-	4050 3400 4150 3400
-Wire Wire Line
-	3850 3100 4050 3100
-Wire Wire Line
-	2750 3950 2700 3950
-Wire Wire Line
-	2700 3950 2700 4000
-Wire Wire Line
 	2850 4550 2700 4550
 Wire Wire Line
@@
 NoConn ~ 8650 2400
 NoConn ~ 9500 5000
+$Comp
+L D D7
+U 1 1 5B31642E
+P 2700 4150
+F 0 "D7" H 2700 4250 50  0000 C CNN
+F 1 "SS14" H 2700 4050 50  0000 C CNN
+F 2 "Diode_SMD:D_SMA" H 2700 4150 50  0001 C CNN
+F 3 "" H 2700 4150 50  0001 C CNN
+	1    2700 4150
+	0    -1   -1   0
+$EndComp
+$Comp
+L D D8
+U 1 1 5B31734F
+P 4050 3100
+F 0 "D8" H 4050 3200 50  0000 C CNN
+F 1 "SS14" H 4050 3000 50  0000 C CNN
+F 2 "Diode_SMD:D_SMA" H 4050 3100 50  0001 C CNN
+F 3 "" H 4050 3100 50  0001 C CNN
+	1    4050 3100
+	1    0    0    -1
+$EndComp
+Wire Wire Line
+	3900 3100 3850 3100
+$Comp
+L R R23
+U 1 1 5B318A76
+P 4200 2900
+F 0 "R23" V 4280 2900 50  0000 C CNN
+F 1 "4k7" V 4200 2900 50  0000 C CNN
+F 2 "Resistor_SMD:R_0603_1608Metric_Pad0.84x1.00mm_HandSolder" V 4130 2900 50  0001 C CNN
+F 3 "" H 4200 2900 50  0001 C CNN
+	1    4200 2900
+	1    0    0    -1
+$EndComp
+Wire Wire Line
+	4200 3050 4200 3100
+Wire Wire Line
+	4200 3100 4300 3100
+Connection ~ 4200 3100
+$Comp
+L VCC #PWR039
+U 1 1 5B31955D
+P 4200 2700
+F 0 "#PWR039" H 4200 2550 50  0001 C CNN
+F 1 "VCC" H 4200 2850 50  0000 C CNN
+F 2 "" H 4200 2700 50  0001 C CNN
+F 3 "" H 4200 2700 50  0001 C CNN
+	1    4200 2700
+	-1   0    0    -1
+$EndComp
+Wire Wire Line
+	4200 2700 4200 2750
 $EndSCHEMATC

Commit message: fix PCB 220v socket
Parts:
- removed D6: SS14, Diode_SMD:D_SMA-SMB_Universal_Handsoldering, symbol D_Schottky
- added R24: 4k7, Resistor_SMD:R_0603_1608Metric_Pad0.84x1.00mm_HandSolder, symbol R
- D5: value MM3Z3V6 -> 5V suppressor
Connections:
- wire segments 200 -> 203
Other:
- moved on the sheet: R27

Commit message: partially worked microdrill
Parts:
- added C14, C15: 0.01 600V, Capacitor_THT:C_Disc_D6.0mm_W2.5mm_P5.00mm, symbol socket-rescue:C
- added R34, R35: 330 2W, Resistor_THT:R_Axial_Power_L20.0mm_W6.4mm_P25.40mm, symbol socket-rescue:R
- C1, C10, C11, C12, C13, C2, C3, C4, C5, C6, C7, C8, C9: symbol C -> socket-rescue:C
- D1: symbol SP0504BAHT -> socket-rescue:SP0504BAHT
- D2: symbol D_Schottky -> socket-rescue:D_Schottky
- D3, D4: symbol BT137-600E -> bt137:BT137-600E
- D5: symbol D_Zener -> socket-rescue:D_Zener
- D7, D8: symbol D -> socket-rescue:D
- J1: symbol DB9_Female -> socket-rescue:DB9_Female
- J2: symbol USB_B -> socket-rescue:USB_B
- J3: symbol Conn_01x02 -> socket-rescue:Conn_01x02
- J4: symbol Conn_01x03 -> socket-rescue:Conn_01x03
- J5: symbol DB15_Male -> socket-rescue:DB15_Male
- J6, J7: symbol Screw_Terminal_01x03 -> socket-rescue:Screw_Terminal_01x03
- K1, K2: symbol G5LE-1 -> socket-rescue:G5LE-1
- Q1, Q2, Q3, Q4, Q5, Q7, Q8, Q9: symbol Q_NMOS_GSD -> socket-rescue:Q_NMOS_GSD
- Q6: symbol Q_PMOS_GSD -> socket-rescue:Q_PMOS_GSD
- R1, R10, R11, R12, R13, R14, R15, R16, R17, R18, R2, R23, R24, R25, R26, R27, R28, R29, R3, R30, R31, R32, R33, R4, R5, R6, R7, R8, R9: symbol R -> socket-rescue:R
- R19, R21: footprint Resistor_THT:R_Axial_DIN0309_L9.0mm_D3.2mm_P12.70mm_Horizontal -> Resistor_SMD:R_1206_HandSoldering; symbol R -> socket-rescue:R
- R20, R22: footprint Resistor_SMD:R_1206_3216Metric_Pad1.24x1.80mm_HandSolder -> Resistor_SMD:R_1206_HandSoldering; symbol R -> socket-rescue:R
- U1: symbol MAX3232 -> socket-rescue:MAX3232
- U10: symbol ACS712 -> acs712:ACS712
- U2: symbol CH340G -> ch34x:CH340G
- U3: symbol STM8S003F3P-RESCUE-socket -> socket-rescue:STM8S003F3P-RESCUE-socket
- U5, U6, U7: symbol PC817 -> socket-rescue:PC817
- U8, U9: symbol MOC3063M -> socket-rescue:MOC3063M
- Y1: symbol Crystal -> socket-rescue:Crystal
Connections:
- net labels added: NC1, NC2
- net labels removed: GNDREF
- wire segments 203 -> 252
- no-connect marks 22 -> 20
